File: pcbs/dust.kicad_pcb (KiCad board)
At the start: 2 copper layers, 113 x 88.2 mm, 43 parts

Commit message: slight changes to pcb
Parts:
- added kibuzzard-6383179D: G***, kibuzzard-6383179D, F.Cu at (267.9, 139.5)
- added kibuzzard-6383179D: G***, kibuzzard-6383179D, B.Cu at (267.9, 139.5)
